File: ZtH/PCB Design/servo_controller_555/servo_controller_555.kicad_sch (KiCad schematic)
At the start: 16 parts, among them J1 SERVO, J2 VIN, U1 LM555xN, U2 AMS1117

Commit message: updated pcb
Parts:
- added TP1, TP2, TP3, TP4, TP5: TestPoint, symbol Connector:TestPoint
Connections:
- net +12V: now also TP1.1
- net +5V: now also TP2.1
- net GND: now also TP3.1
- net at J1.3 (Pin_3), U1.3 (OUT): now also TP5.1
- net at C1.1, D1.1 (K), R1.1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: now also TP4.1
Other:
- moved on the sheet: C2
