File: ZtH/PCB Design/servo_controller_555/servo_controller_555.kicad_pcb (KiCad board)
At the start: 2 copper layers, 60 x 50 mm, 23 parts, among them J1 SERVO, J2 VIN, U1 LM555xN, U2 AMS1117

Commit message: PCB and Lab Tools Complete
Routing:
- net +5V: track 121.2 -> 117.4 mm
Other:
- board text added: "+"
- board text added: "+12v"
- board text added: "+5v"
- board text added: "-"
- board text added: "NU Teams 555 Servo Driver v1 Theo Devos-Vernes c3479858 15/08/2026"
- board text added: "SIG"
- board text removed: "NU Teams 555 Servo Driver v1"
- board text removed: "Theo Devos-Vernes c3479858 15/08/2026"
Changed lines of the file:
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@@
 		(tags "THT DIP DIL PDIP 2.54mm 7.62mm 300mil")
 		(property "Reference" "U1"
-			(at 0 -2.42 0)
+			(at 0 -1.92 0)
 			(layer "F.SilkS")
 			(effects
@@
 		)
 		(fp_text user "K"
-			(at -0.88 1.92 0)
+			(at 0.12 1.92 0)
 			(layer "F.SilkS")
 			(effects
@@
 		(tags "LED handsolder")
 		(property "Reference" "D3"
-			(at -0.025 -2 0)
+			(at 3.475 0 0)
 			(layer "F.SilkS")
 			(effects
@@
 		(tags "LED")
 		(property "Reference" "D2"
-			(at 1.27 -3.96 0)
+			(at 5.54 0 0)
 			(layer "F.SilkS")
 			(effects
@@
 		(layer "Edge.Cuts")
 	)
-	(gr_text "Theo Devos-Vernes\nc3479858\n15/08/2026"
-		(at 59.5 66 0)
+	(gr_text "+"
+		(at 51.28 91 0)
 		(layer "F.SilkS")
 		(effects
 			(font
 				(size 1 1)
-				(thickness 0.1)
+				(thickness 0.2)
+				(bold yes)
 			)
 			(justify left bottom)
 		)
 	)
-	(gr_text "NU Teams 555 Servo Driver v1"
-		(at 77.5 63 0)
+	(gr_text "-"
+		(at 51.5 78 0)
 		(layer "F.SilkS")
 		(effects
 			(font
 				(size 1 1)
-				(thickness 0.1)
+				(thickness 0.2)
+				(bold yes)
+			)
+			(justify left bottom)
+		)
+	)
+	(gr_text "+5v"
+		(at 66 68.5 0)
+		(layer "F.SilkS" knockout)
+		(effects
+			(font
+				(size 1 1)
+				(thickness 0.2)
+				(bold yes)
+			)
+			(justify left bottom)
+		)
+	)
+	(gr_text "+12v"
+		(at 66 97.5 0)
+		(layer "F.SilkS" knockout)
+		(effects
+			(font
+				(size 1 1)
+				(thickness 0.2)
+				(bold yes)
+			)
+			(justify left bottom)
+		)
+	)
+	(gr_text "NU Teams 555 Servo Driver v1\nTheo Devos-Vernes\nc3479858\n15/08/2026"
+		(at 77.5 68 0)
+		(layer "F.SilkS")
+		(effects
+			(font
+				(size 1 1)
+				(thickness 0.2)
+				(bold yes)
+			)
+			(justify left bottom)
+		)
+	)
+	(gr_text "-"
+		(at 107 83 0)
+		(layer "F.SilkS")
+		(effects
+			(font
+				(size 1 1)
+				(thickness 0.2)
+				(bold yes)
+			)
+			(justify left bottom)
+		)
+	)
+	(gr_text "+"
+		(at 107 85.5 0)
+		(layer "F.SilkS")
+		(effects
+			(font
+				(size 1 1)
+				(thickness 0.2)
+				(bold yes)
+			)
+			(justify left bottom)
+		)
+	)
+	(gr_text "SIG"
+		(at 107 88.5 0)
+		(layer "F.SilkS")
+		(effects
+			(font
+				(size 1 1)
+				(thickness 0.2)
+				(bold yes)
 			)
 			(justify left bottom)
@@
 	)
 	(segment
-		(start 100 85)
-		(end 100 78.5)
-		(width 0.4)
-		(layer "F.Cu")
-		(net "+5V")
-	)
-	(segment
 		(start 87.88 93.08)
 		(end 87.88 95.08)
@@
 	)
 	(segment
-		(start 80 70)
-		(end 73 77)
-		(width 0.4)
-		(layer "F.Cu")
-		(net "+5V")
-	)
-	(segment
 		(start 87.88 95.08)
 		(end 90.38 97.58)
@@
 	)
 	(segment
-		(start 91.5 70)
-		(end 80 70)
-		(width 0.4)
-		(layer "F.Cu")
-		(net "+5V")
-	)
-	(segment
 		(start 68.5375 82.0375)
 		(end 71.5 85)
@@
 	)
 	(segment
-		(start 105 85)
-		(end 100 85)
+		(start 104.75 85)
+		(end 89.75 70)
 		(width 0.4)
 		(layer "F.Cu")
@@
 	)
 	(segment
-		(start 65.2 85)
-		(end 71.5 85)
+		(start 89.75 70)
+		(end 80 70)
+		(width 0.4)
+		(layer "F.Cu")
+		(net "+5V")
+	)
+	(segment
+		(start 80 70)
+		(end 73 77)
+		(width 0.4)
+		(layer "F.Cu")
+		(net "+5V")
+	)
+	(segment
+		(start 105 85)
+		(end 104.75 85)
 		(width 0.4)
 		(layer "F.Cu")
@@
 	)
 	(segment
-		(start 100 78.5)
-		(end 91.5 70)
+		(start 65.2 85)
+		(end 71.5 85)
 		(width 0.4)
 		(layer "F.Cu")

Commit message: finish pcb frfr ong
Parts:
- added +12V: TestPoint, TestPoint:TestPoint_THTPad_D2.0mm_Drill1.0mm, F.Cu at (60.0, 99.0)
- added +5V: TestPoint, TestPoint:TestPoint_THTPad_D2.0mm_Drill1.0mm, F.Cu at (77.0, 85.0)
- added GND: TestPoint, TestPoint:TestPoint_Pad_4.0x4.0mm, B.Cu at (63.5, 107.5)
- added SIG: TestPoint, TestPoint:TestPoint_THTPad_D2.0mm_Drill1.0mm, F.Cu at (106.0, 94.0)
- added TP4: TestPoint, TestPoint:TestPoint_THTPad_D2.0mm_Drill1.0mm, F.Cu at (102.0, 97.0)
- moved G*** 14.7 mm to (67.5, 90.5)
- moved ThinkFast 14.7 mm to (67.5, 83.5)
Routing:
- net Net-(D1-K): track 23.1 -> 31.1 mm
- net Net-(J1-Pin_3): track 9.69 -> 16.3 mm
- net +12V: track 17.6 -> 23.3 mm
- net +5V: track 117.4 -> 122.9 mm

Commit message: ok pcb finished fr fr fr fr fr ong fr ong ong fr
Parts:
- moved G*** 33.4 mm to (99.0, 79.5)
- moved ThinkFast 33.4 mm to (99.0, 72.5)
- moved J1 3.00 mm to (108.0, 82.5)
- moved J2 0.50 mm to (55.5, 81.5)
Routing:
- net Net-(J1-Pin_3): track 16.3 -> 19.9 mm
- net +5V: track 122.9 -> 125.9 mm
Other:
- board text added: "7-12Vin"
Changed lines of the file:
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@@
 				(font
 					(size 1 1)
-					(thickness 0.15)
+					(thickness 0.2)
+					(bold yes)
 				)
 			)
@@
 	(footprint "Connector_PinHeader_2.54mm:PinHeader_1x03_P2.54mm_Vertical"
 		(layer "F.Cu")
-		(at 105 82.46)
+		(at 108 82.5)
 		(descr "Through hole straight pin header, 1x03, 2.54mm pitch, single row")
 		(tags "Through hole pin header THT 1x03 2.54mm single row")
@@
 	(footprint "TerminalBlock_Phoenix:TerminalBlock_Phoenix_MKDS-1,5-2_1x02_P5.00mm_Horizontal"
 		(layer "F.Cu")
-		(at 56 81.5 -90)
+		(at 55.5 81.5 -90)
 		(descr "Terminal Block Phoenix MKDS-1,5-2, 2 pins, pitch 5mm, size 10x9.8mm, drill diameter 1.3mm, pad diameter 2.6mm, http://www.farnell.com/datasheets/100425.pdf")
 		(tags "THT Terminal Block Phoenix MKDS-1,5-2 pitch 5mm size 10x9.8mm drill 1.3mm pad 2.6mm")
@@
 				(font
 					(size 1 1)
-					(thickness 0.2)
-					(bold yes)
+					(thickness 0.125)
 				)
 				(justify mirror)
@@
 	(footprint "LOGO"
 		(layer "B.Cu")
-		(at 67.5 83.5 180)
+		(at 99 72.5 180)
 		(property "Reference" "ThinkFast"
 			(at -4 5 0)
@@
 	(footprint "LOGO"
 		(layer "B.Cu")
-		(at 67.5 90.5 180)
+		(at 99 79.5 180)
 		(property "Reference" "G***"
 			(at 0 0 0)
@@
 		(layer "Edge.Cuts")
 	)
+	(gr_text "7-12Vin"
+		(at 50.5 91 270)
+		(layer "F.SilkS")
+		(effects
+			(font
+				(size 1 1)
+				(thickness 0.1)
+			)
+			(justify left bottom)
+		)
+	)
 	(gr_text "+"
 		(at 51.28 91 0)
@@
 		)
 	)
-	(gr_text "-"
-		(at 107 83 0)
+	(gr_text "SIG"
+		(at 104 88.5 0)
 		(layer "F.SilkS")
 		(effects
@@
 		)
 	)
-	(gr_text "+"
-		(at 107 85.5 0)
+	(gr_text "-"
+		(at 105 83 0)
 		(layer "F.SilkS")
 		(effects
@@
 		)
 	)
-	(gr_text "SIG"
-		(at 107 88.5 0)
+	(gr_text "+"
+		(at 105 85.5 0)
 		(layer "F.SilkS")
 		(effects
@@
 	)
 	(segment
-		(start 95.5 88)
-		(end 104.54 88)
+		(start 108 92)
+		(end 108 87.58)
 		(width 0.2)
 		(layer "F.Cu")
@@
 	)
 	(segment
-		(start 104.54 88)
-		(end 105 87.54)
+		(start 95.5 88)
+		(end 107.58 88)
 		(width 0.2)
 		(layer "F.Cu")
@@
 	)
 	(segment
-		(start 106 94)
-		(end 104.54 92.54)
+		(start 107.58 88)
+		(end 108 87.58)
 		(width 0.2)
 		(layer "F.Cu")
@@
 	)
 	(segment
-		(start 104.54 92.54)
-		(end 104.54 88)
+		(start 106 94)
+		(end 108 92)
 		(width 0.2)
 		(layer "F.Cu")
@@
 	)
 	(segment
+		(start 73 77)
+		(end 68.5375 77)
+		(width 0.4)
+		(layer "F.Cu")
+		(net "+5V")
+	)
+	(segment
 		(start 68.5375 77)
 		(end 69 76.5375)
@@
 	)
 	(segment
+		(start 108 85.04)
+		(end 92.96 70)
+		(width 0.4)
+		(layer "F.Cu")
+		(net "+5V")
+	)
+	(segment
 		(start 87.88 93.08)
 		(end 87.88 95.08)
@@
 	)
 	(segment
+		(start 80 70)
+		(end 73 77)
+		(width 0.4)
+		(layer "F.Cu")
+		(net "+5V")
+	)
+	(segment
 		(start 68.5375 77)
 		(end 68.5375 82.0375)
@@
 	)
 	(segment
-		(start 104.75 85)
-		(end 89.75 70)
-		(width 0.4)
-		(layer "F.Cu")
-		(net "+5V")
-	)
-	(segment
-		(start 89.75 70)
+		(start 92.96 70)
 		(end 80 70)
 		(width 0.4)
@@
 	)
 	(segment
-		(start 80 70)
-		(end 73 77)
-		(width 0.4)
-		(layer "F.Cu")
-		(net "+5V")
-	)
-	(segment
-		(start 105 85)
-		(end 104.75 85)
-		(width 0.4)
-		(layer "F.Cu")
-		(net "+5V")
-	)
-	(segment
 		(start 65.2 85)
 		(end 71.5 85)
@@
 	)
 	(segment
-		(start 73 77)
-		(end 68.5375 77)
-		(width 0.4)
-		(layer "F.Cu")
-		(net "+5V")
-	)
-	(segment
 		(start 78.1 94.56)
 		(end 79.58 93.08)
@@
 	)
 	(segment
-		(start 54.5 93.5)
-		(end 56 92)
+		(start 55.5 86.5)
+		(end 55.5 92.5)
 		(width 0.4)
 		(layer "F.Cu")
@@
 	)
 	(segment
-		(start 56 92)
-		(end 56 86.5)
+		(start 55.5 92.5)
+		(end 54.5 93.5)
 		(width 0.4)
 		(layer "F.Cu")
