File: DRS Project/Design Files/Electrical System/DRS_Control_Unit/DRS_Control_Unit.kicad_sch (KiCad schematic)
At the start: 0 parts

Commit message: power system started
Parts:
- added C1: 110u (CHANGE REQ), Package_TO_SOT_SMD:SOT-23-6, symbol Device:C_Polarized
- added C2: 220u (CHANGE REQ), Package_TO_SOT_SMD:SOT-23-6, symbol Device:C_Polarized
- added C3: FF, Package_TO_SOT_SMD:SOT-23-6, symbol Device:C
- added D1: 1N5822, Diode_THT:D_DO-201AD_P15.24mm_Horizontal, symbol Diode:1N5822
- added D2: D, symbol Device:D
- added J1: TEMP VIN, Package_SO:MSOP-16-1EP_3x4.039mm_P0.5mm_EP1.651x2.845mm_ThermalVias, symbol Connector:Screw_Terminal_01x02
- added L1: 33u, symbol Device:L
- added R1: 1.0k, symbol Device:R
- added R2: 3.1k, symbol Device:R
- added U1: LM2596S-5, Package_TO_SOT_SMD:TO-263-5_TabPin3, symbol Regulator_Switching:LM2596S-5
Connections:
- new net: C3.1, R1.2, R2.1, U1.4 (FB)
- new net: D2.2 (A), J1.2 (Pin_2)
- new net: D1.1 (K), L1.1, U1.2 (OUT)
- new net +12-14V: C1.1, D2.1 (K), U1.1 (VIN)
- new net +5V: C2.1, C3.2, L1.2, R2.2
- new net GND: C1.2, C2.2, D1.2 (A), J1.1 (Pin_1), R1.1, U1.3 (GND), U1.5 (~{ON}/OFF)
Other:
- note added: "Power Input and Regulation"

Commit message: improved kicad model
Parts:
- removed J1: TEMP VIN, Package_SO:MSOP-16-1EP_3x4.039mm_P0.5mm_EP1.651x2.845mm_ThermalVias, symbol Connector:Screw_Terminal_01x02
- added D3: UNFUSED, symbol Device:LED
- added D4: FUSED, symbol Device:LED
- added D5: PROTEC, symbol Device:LED
- added D6: REGULATED, symbol Device:LED
- added F1: 5A, Package_LCC:PLCC-84_29.3x29.3mm_P1.27mm, symbol Device:Fuse
- added J1: Deutsch DT, Package_DFN_QFN:QFN-20-1EP_5x5mm_P0.65mm_EP3.35x3.35mm, symbol Connector:Conn_01x06_Pin
- added R3, R4, R5, R6: R, symbol Device:R
- added U2: TJA1051T-3, Package_SO:SOIC-8_3.9x4.9mm_P1.27mm, symbol Interface_CAN_LIN:TJA1051T-3
- added U3: DEV-15583, DEV-15583:MODULE_DEV-15583, symbol DEV-15583:DEV-15583
- C1: value 110u (CHANGE REQ) -> 110u
- C2: value 220u (CHANGE REQ) -> 220u
- C3: value FF -> 5n
- D2: value D -> MUST HOLD REVERSE CURRENT
- R2: value 3.1k -> 3.3k
Connections:
- net GND: now also J1.2 (Pin_2), J1.5 (Pin_5), R3.2, R4.2, R5.2, R6.1, U2.2 (GND), U2.8 (S), U3.G1
- net at D2.2 (A): now also D4.2 (A), F1.2
- net +12-14V renamed +12V
- net +12V: now also D3.2 (A), D5.2 (A), F1.1, J1.1 (Pin_1), J1.6 (Pin_6)
- net +5V renamed +5.5V
- net +5.5V: now also D6.2 (A), U2.3 (VCC), U2.5 (VIO), U3.VIN
- new net: D6.1 (K), R6.2
- new net: D4.1 (K), R4.1
- new net: D3.1 (K), R3.1
- new net: D5.1 (K), R5.1
- new net CAN HIGH: J1.4 (Pin_4), U2.7 (CANH)
- new net CAN LOW: J1.3 (Pin_3), U2.6 (CANL)
- new net RX: U2.4 (RXD), U3.0
- new net TX: U2.1 (TXD), U3.1
Other:
- note added: "Expansion Port"
- note added: "Power Input and Regulation (WIP)"
- note removed: "Power Input and Regulation"
- moved on the sheet: C1, C2, C3, D1, D2, L1, R1, R2, U1

Commit message: updated control unit
Connections:
- net +12V: no longer C1.1, D2.1 (K), D5.2 (A), U1.1 (VIN)
- net +5.5V: no longer U2.5 (VIO)
- net GND: now also U3.G2
- net RX: no longer names the net of U2.4 (RXD), U3.0
- net TX: no longer names the net of U2.1 (TXD), U3.1
- new net: C1.1, D2.1 (K), D5.2 (A), U1.1 (VIN)
- no-connect marks 0 -> 29
Other:
- moved on the sheet: U2, U3

Commit message: updated control unit
Parts:
- U3: footprint DEV-15583:MODULE_DEV-15583 -> TEENSY_4:MODULE_DEV-15583
Changed lines of the file:
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@@
 	)
 	(junction
-		(at 63.5 99.06)
+		(at 68.58 109.22)
 		(diameter 0)
 		(color 0 0 0 0)
@@
 	(wire
 		(pts
+			(xy 68.58 96.52) (xy 68.58 109.22)
+		)
+		(stroke
+			(width 0)
+			(type default)
+		)
+	)
+	(wire
+		(pts
 			(xy 43.18 91.44) (xy 44.45 91.44)
 		)
@@
 	(wire
 		(pts
-			(xy 68.58 96.52) (xy 68.58 99.06)
-		)
-		(stroke
-			(width 0)
-			(type default)
-		)
-	)
-	(wire
-		(pts
 			(xy 54.61 106.68) (xy 54.61 109.22)
 		)
@@
 	(wire
 		(pts
-			(xy 63.5 109.22) (xy 81.28 109.22)
+			(xy 63.5 109.22) (xy 68.58 109.22)
 		)
 		(stroke
@@
 	(wire
 		(pts
-			(xy 63.5 99.06) (xy 68.58 99.06)
-		)
-		(stroke
-			(width 0)
-			(type default)
-		)
-	)
-	(wire
-		(pts
 			(xy 39.37 33.02) (xy 39.37 41.91)
 		)
@@
 		(pts
 			(xy 123.19 96.52) (xy 124.46 96.52)
+		)
+		(stroke
+			(width 0)
+			(type default)
+		)
+	)
+	(wire
+		(pts
+			(xy 68.58 109.22) (xy 81.28 109.22)
 		)
 		(stroke
@@
 			)
 		)
-		(property "Footprint" "DEV-15583:MODULE_DEV-15583"
+		(property "Footprint" "TEENSY_4:MODULE_DEV-15583"
 			(at 195.58 83.82 0)
 			(hide yes)

Commit message: finished v1 of circuit board
Parts:
- removed D1: 1N5822, Diode_THT:D_DO-201AD_P15.24mm_Horizontal, symbol Diode:1N5822
- removed D2: MUST HOLD REVERSE CURRENT, symbol Device:D
- removed U1: LM2596S-5, Package_TO_SOT_SMD:TO-263-5_TabPin3, symbol Regulator_Switching:LM2596S-5
- added D1, D2, D7: SS54, Package_SON:WSON-8-1EP_6x5mm_P1.27mm_EP3.4x4mm, symbol Device:D_Schottky
- added J2: Servo, Package_DFN_QFN:QFN-20-1EP_5x5mm_P0.65mm_EP3.35x3.35mm, symbol Connector:Conn_01x03_Pin
- added U1: LM2596S-ADJ, Package_TO_SOT_SMD:TO-263-5_TabPin3, symbol Regulator_Switching:LM2596S-ADJ
- C1: value 110u -> 100u
- D3, D4, D5, D6: footprint (none) -> LED_SMD:LED_1206_3216Metric_Pad1.42x1.75mm_HandSolder
- R1, R2: footprint (none) -> Resistor_SMD:R_1206_3216Metric_Pad1.30x1.75mm_HandSolder
- R3, R4, R5: value R -> 1.2k; footprint (none) -> Resistor_SMD:R_1206_3216Metric_Pad1.30x1.75mm_HandSolder
- R6: value R -> 330r; footprint (none) -> Resistor_SMD:R_1206_3216Metric_Pad1.30x1.75mm_HandSolder
- U3: value DEV-15583 -> TEENSY 4.0
Connections:
- net GND: now also U3.G3, D1.2 (A), J2.1 (Pin_1), U1.3 (GND), U1.5 (~{ON}/OFF)
- net SIGNAL: now reaches U3.2
- net SIGNAL: now also J2.3 (Pin_3)
- net at C3.1, R1.2, R2.1: now also U1.4 (FB)
- net at C1.1, D5.2 (A): now also D2.1 (K), U1.1 (VIN)
- net at L1.1: now also D1.1 (K), U1.2 (OUT)
- net at D4.2 (A), F1.2: now also D2.2 (A)
- net +5.5V renamed +5.3V
- net +5.3V: now also D7.2 (A), J2.2 (Pin_2); no longer U3.VIN
- new net: D7.1 (K), U3.VIN
- no-connect marks 29 -> 27
Other:
- note added: "Power Input and Regulation"
- note added: "Servo Output"
- note added: "Teensy 4.0 + CAN Transceiver"
- note removed: "Power Input and Regulation (WIP)"
- moved on the sheet: C1, C2, C3, D3, D4, D5, D6, F1, J1, L1, R1, R2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

Commit message: v1 of circuit diagram complete
Parts:
- added TP1: UNFUS, symbol Connector:TestPoint
- added TP2: FUSED, symbol Connector:TestPoint
- added TP3: GND, symbol Connector:TestPoint
- added TP4: +5.3V, symbol Connector:TestPoint
- added TP5: CANH, symbol Connector:TestPoint
- added TP6: CANL, symbol Connector:TestPoint
Connections:
- net +12V: now also TP1.1
- net +5.3V: now also TP4.1
- net CAN HIGH: now also TP5.1
- net CAN LOW: now also TP6.1
- net GND: now also TP3.1
- net at C1.1, D2.1 (K), D5.2 (A)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: now also TP2.1
Other:
- company: (none) -> NU Teams
- title: (none) -> DRS Control Unit
- moved on the sheet: C1, C2, C3, D1, D2, D3, D4, D5, D6, D7, F1, J1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

Commit message: updated
Parts:
- F1: footprint Package_LCC:PLCC-84_29.3x29.3mm_P1.27mm -> (none)
- L1: footprint (none) -> DRS_Library:Inductor_HCM1A1104V3
- TP1, TP2, TP3, TP4, TP5, TP6: footprint (none) -> TestPoint:TestPoint_THTPad_D2.0mm_Drill1.0mm
Changed lines of the file:
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@@
 			)
 		)
-		(property "Footprint" ""
+		(property "Footprint" "TestPoint:TestPoint_THTPad_D2.0mm_Drill1.0mm"
 			(at 257.81 146.05 0)
 			(hide yes)
@@
 			)
 		)
-		(property "Footprint" ""
+		(property "Footprint" "TestPoint:TestPoint_THTPad_D2.0mm_Drill1.0mm"
 			(at 181.61 57.15 0)
 			(hide yes)
@@
 			)
 		)
-		(property "Footprint" "Package_LCC:PLCC-84_29.3x29.3mm_P1.27mm"
+		(property "Footprint" ""
 			(at 181.61 58.928 90)
 			(hide yes)
@@
 			)
 		)
-		(property "Footprint" ""
+		(property "Footprint" "DRS_Library:Inductor_HCM1A1104V3"
 			(at 246.38 62.23 0)
 			(hide yes)
@@
 			)
 		)
-		(property "Footprint" ""
+		(property "Footprint" "TestPoint:TestPoint_THTPad_D2.0mm_Drill1.0mm"
 			(at 271.78 62.23 0)
 			(hide yes)
@@
 			)
 		)
-		(property "Footprint" ""
+		(property "Footprint" "TestPoint:TestPoint_THTPad_D2.0mm_Drill1.0mm"
 			(at 267.97 140.97 0)
 			(hide yes)
@@
 			)
 		)
-		(property "Footprint" ""
+		(property "Footprint" "TestPoint:TestPoint_THTPad_D2.0mm_Drill1.0mm"
 			(at 207.01 74.93 0)
 			(hide yes)
@@
 			)
 		)
-		(property "Footprint" ""
+		(property "Footprint" "TestPoint:TestPoint_THTPad_D2.0mm_Drill1.0mm"
 			(at 212.09 57.15 0)
 			(hide yes)

Commit message: MORE updates to design files
Parts:
- removed U3: TEENSY 4.0, TEENSY_4:MODULE_DEV-15583, symbol DEV-15583:DEV-15583
- added U3: Teensy4.0-NU-Teams, NU-Teams-Footprints:Teensy4.0-NU-Teams, symbol NU-Teams-KiCAD-Library:Teensy4.0-NU-Teams
- D1, D2, D7: footprint Package_SON:WSON-8-1EP_6x5mm_P1.27mm_EP3.4x4mm -> (none)
- J1: footprint Package_DFN_QFN:QFN-20-1EP_5x5mm_P0.65mm_EP3.35x3.35mm -> NU-Teams-Footprints:DT15-6P
- J2: footprint Package_DFN_QFN:QFN-20-1EP_5x5mm_P0.65mm_EP3.35x3.35mm -> Connector_PinHeader_2.54mm:PinHeader_1x03_P2.54mm_Vertical
Connections:
- net GND: now also U3.GNDB (GND), U3.GNDL (GND), U3.GNDR (GND)
- net SIGNAL: now also U3.2 (2_OUT2)
- net at U2.4 (RXD): now also U3.0 (0_CAN2_RX)
- net at U2.1 (TXD): now also U3.1 (1_CAN2_TX)
- net at D7.1 (K): now also U3.VIN
- net +5.3V renamed +6V
Other:
- moved on the sheet: C1, C2, C3, D1, D2, D3, D4, D5, D6, D7, F1, J1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
