File: DRS Project/Design Files/Electrical System/DRS_Control_Unit/DRS_Control_Unit.kicad_sch (KiCad schematic)
At the start: 47 parts, among them IC1 AP63301QWU-7, J1 Screw, J2 Deutsch DT, J3 Servo, J4 DE9_Socket, SW1 DSIC01THGET, U1 AMS1117, U2 Teensy4.0-NU-Teams, U3 TJA1051T-3, U4 LM2596S-ADJ

Commit message: improved PCB design (still unfinished)
Parts:
- removed J4: DE9_Socket, Connector_Dsub:DSUB-9_Socket_Vertical_P2.77x2.84mm, symbol Connector:DE9_Socket
- added J4: DE9_Socket_MountingHoles, Connector_Dsub:DSUB-9_Socket_Vertical_P2.77x2.84mm_MountingHoles, symbol Connector:DE9_Socket_MountingHoles
- J1: footprint NU-Teams-Footprints:DT15-6P -> TerminalBlock_Phoenix:TerminalBlock_Phoenix_MKDS-1,5-2_1x02_P5.00mm_Horizontal
- J2: footprint TerminalBlock_Phoenix:TerminalBlock_Phoenix_MKDS-1,5-2_1x02_P5.00mm_Horizontal -> NU-Teams-Footprints:DT15-6P
- R5: footprint Connector_PinSocket_2.54mm:PinSocket_1x02_P2.54mm_Vertical -> Resistor_SMD:R_1206_3216Metric_Pad1.30x1.75mm_HandSolder
- R6: footprint Resistor_SMD:R_1206_3216Metric_Pad1.30x1.75mm_HandSolder -> Connector_PinSocket_2.54mm:PinSocket_1x02_P2.54mm_Vertical
Connections:
- net CAN HIGH: now also J4.7
- net CAN LOW: now also J4.2
- no-connect marks 34 -> 35

Commit message: pcb rev 1 actually complete (fr this time)
Parts:
- added D8: +(VAR)V U.F., LED_SMD:LED_1206_3216Metric_Pad1.42x1.75mm_HandSolder, symbol Device:LED
- added D9: +(VAR)V F, LED_SMD:LED_1206_3216Metric_Pad1.42x1.75mm_HandSolder, symbol Device:LED
- added R10, R11: 680R, Resistor_SMD:R_1206_3216Metric_Pad1.30x1.75mm_HandSolder, symbol Device:R
- added TP3: +5V Regulated., TestPoint:TestPoint_Loop_D1.80mm_Drill1.0mm_Beaded, symbol Connector:TestPoint
- added TP4: +12V Fused, TestPoint:TestPoint_Loop_D1.80mm_Drill1.0mm_Beaded, symbol Connector:TestPoint
- added TP5: Ground, TestPoint:TestPoint_Loop_D1.80mm_Drill1.0mm_Beaded, symbol Connector:TestPoint
- added TP6: Servo Signal, TestPoint:TestPoint_Loop_D1.80mm_Drill1.0mm_Beaded, symbol Connector:TestPoint
- added TP7: +(VAR)V Regulated, TestPoint:TestPoint_Loop_D1.80mm_Drill1.0mm_Beaded, symbol Connector:TestPoint
- J4: value DE9_Socket_MountingHoles -> DE-9 Socket
- renumbered C8 to C1, C7 to C10, C9 to C2, C10 to C3, C1 to C4, C2 to C5, C3 to C6, C4 to C7, C5 to C8, C6 to C9, D6 to D1, D7 to D2, D1 to D3, D2 to D4, D3 to D5, D4 to D6, D5 to D7, F3 to F1, F1 to F2, F2 to F3, J3 to J2, J2 to J3, L2 to L1, L1 to L2, R9 to R1, R7 to R12, R8 to R13, R10 to R2, R11 to R3, R1 to R4, R2 to R5, R3 to R6, R4 to R7, R5 to R8, R6 to R9, TP3 to TP1, TP4 to TP2, TP1 to TP8, TP2 to TP9, U4 to U1, U1 to U2, U2 to U3, U3 to U4
Connections:
- net +(VAR)V: now also D9.2 (A), TP7.1
- net GND: now also R10.1, R11.2, TP5.1
- net SIGNAL: now also TP6.1
- net VIN: now also TP4.1
- net at C4.1, D3.2 (A), D6.2 (A)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: now also TP3.1
- net at C6.2, C7.1, F3.1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: now also D8.2 (A)
- new net: D9.1 (K), R11.1
- new net: D8.1 (K), R10.2
Other:
- moved on the sheet: C1, C10, C2, C3, C4, C5, C6, C7, C8, C9, D1, D2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

Commit message: improved pcb design (unfinished)
Changed lines of the file:
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@@
 		)
 	)
-	(text_box "Non standard block. Reason for using this over a standard circuit is that this power regulation circuit can deliver the required current to our servo, whereas standard servo would be overloaded."
+	(text_box "Non standard block. Reason for using this over a standard circuit is that this power regulation circuit can deliver the required current to our servo, whereas standard buck converter circuit would be overloaded."
 		(exclude_from_sim no)
 		(at 29.21 106.68 0)
@@
 		)
 	)
-	(text_box "Non standard block. Reason is for space efficiency compared to standard +5V regulation circuit."
+	(text_box "Non standard block. Reason is for space efficiency compared to standard 5V regulation circuit."
 		(exclude_from_sim no)
 		(at 80.01 53.34 0)

Commit message: made minor changes to pcb and *nearly* finished
Parts:
- removed D3: SS34, Diode_SMD:D_SMA_Handsoldering, symbol Device:D_Schottky
- removed D6: +5V, LED_SMD:LED_1206_3216Metric_Pad1.42x1.75mm_HandSolder, symbol Device:LED
- added D10: +12V PR, LED_SMD:LED_1206_3216Metric_Pad1.42x1.75mm_HandSolder, symbol Device:LED
- added D6: SS54, Diode_SMD:D_SMA_Handsoldering, symbol Device:D_Schottky
- added U5: Branding_Block_Racing, NU-Teams-Footprints:BRANDING_RACING, symbol NU-Teams-KiCAD-Library:Branding_Block_Racing
- D7: value +5V PROT -> +5V
- F2: value 5A -> 4A
- R6: value 330R -> 1.2k
Connections:
- net +5V: now also C4.1, TP3.1, U2.2 (VO)
- net GND: now also R6.2; no longer R6.1
- net VIN: now also D10.2 (A), D6.1 (K); no longer D5.2 (A), F2.2, TP4.1
- new net: D5.2 (A), D6.2 (A), F2.2, TP4.1
- new net: D10.1 (K), R6.1
Other:
- moved on the sheet: C4, D4, D5, D7, F2, R4, R5, R7, TP4

Commit message: updated
Parts:
- C10: footprint Capacitor_SMD:C_1206_3216Metric -> Capacitor_SMD:C_1206_3216Metric_Pad1.33x1.80mm_HandSolder
- J2: footprint Connector_PinHeader_2.54mm:PinHeader_1x03_P2.54mm_Horizontal -> Connector_PinHeader_2.54mm:PinHeader_1x03_P2.54mm_Vertical
Changed lines of the file:
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@@
 			)
 		)
-		(property "Footprint" "Capacitor_SMD:C_1206_3216Metric"
+		(property "Footprint" "Capacitor_SMD:C_1206_3216Metric_Pad1.33x1.80mm_HandSolder"
 			(at 44.1452 142.24 0)
 			(hide yes)
@@
 			)
 		)
-		(property "Footprint" "Connector_PinHeader_2.54mm:PinHeader_1x03_P2.54mm_Horizontal"
+		(property "Footprint" "Connector_PinHeader_2.54mm:PinHeader_1x03_P2.54mm_Vertical"
 			(at 215.9 123.19 0)
 			(hide yes)

Commit message: PCB DONE WOOOOOOO
Parts:
- added H1, H2, H3, H4: (no value), MountingHole:MountingHole_6.4mm_M6, symbol Mechanical:MountingHole
- U5: value Branding_Block_Racing -> (none)
Other:
- note added: "Mounting Holes & Branding Block"
- moved on the sheet: J1, J2, U5

Commit message: PCB AND SCHEMATIC DONEZO
Parts:
- added TP10: +12V Protected, TestPoint:TestPoint_Loop_D1.80mm_Drill1.0mm_Beaded, symbol Connector:TestPoint
- D10: value +12V PR -> +12V PROT
- D4: value +12V U.F. -> +12V RAW
- D5: value +12V F -> +12V FUSED
- D8: value +(VAR)V U.F. -> +6-8V RAW
- D9: value +(VAR)V F -> +6-8V FUSED
- R12: footprint Resistor_SMD:R_1206_3216Metric -> Resistor_SMD:R_1206_3216Metric_Pad1.30x1.75mm_HandSolder
- R13: value 120 -> 120R
- TP7: value +(VAR)V Regulated -> +6-8V REGULATED
Connections:
- net VIN: now also TP10.1
- net +(VAR)V renamed +6-8V
Other:
- note removed: "Testing Terminal"
- moved on the sheet: C4, C8, D10, D4, D5, D6, D7, F2, H1, H2, H3, H4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

Commit message: Rev1.1 Started
Rev1.1
Connections:
- net +3.3V: now reaches U3.3V3R (3V3)
- net +3.3V: now also U4.5 (VIO)
- no-connect marks 35 -> 33
