File: DRS Project/Design Files/Electrical System/DRS_Control_Unit/DRS_Control_Unit.kicad_pcb (KiCad board)
At the start: 2 copper layers, 100 x 100 mm, 52 parts, among them IC1 AP63301QWU-7, J1 Screw, J2 Servo, J3 Deutsch DT, J4 DE-9 Socket, SW1 DSIC01THGET, U2 AMS1117, U3 Teensy4.0-NU-Teams, U4 TJA1051T-3

Commit message: PCB AND SCHEMATIC DONEZO
Parts:
- added TP10: +12V Protected, TestPoint:TestPoint_Loop_D1.80mm_Drill1.0mm_Beaded, F.Cu at (113.4, 89.9)
- D10: value +12V PR -> +12V PROT
- D4: value +12V U.F. -> +12V RAW
- D5: value +12V F -> +12V FUSED
- D8: value +(VAR)V U.F. -> +6-8V RAW
- D9: value +(VAR)V F -> +6-8V FUSED
- G*** (x2): moved to B.Cu
- R12: footprint Resistor_SMD:R_1206_3216Metric -> Resistor_SMD:R_1206_3216Metric_Pad1.30x1.75mm_HandSolder
- R13: value 120 -> 120R
- TP7: value +(VAR)V Regulated -> +6-8V REGULATED
- moved G*** 18.1 mm to (181.6, 108.2)
- moved TP8 12.3 mm to (173.9, 100.0)
- moved R13 10.7 mm to (167.5, 80.2)
- moved TP9 10.1 mm to (166.5, 100.0)
- moved G*** 9.10 mm to (133.8, 57.0), turned to 180 degrees
- moved SW1 7.67 mm to (173.8, 84.2), turned to 180 degrees
- moved TP5 7.34 mm to (159.6, 100.1)
- moved TP7 5.66 mm to (119.5, 90.4)
- moved G*** 5.18 mm to (140.9, 57.2), turned to 180 degrees
- moved F3 3.00 mm to (123.0, 76.2)
- moved J1 1.40 mm to (95.8, 113.9)
Connections:
- net +(VAR)V renamed +6-8V
Routing:
- net /CAN HIGH: track 107.8 -> 86.5 mm
- net /VIN: track 45.5 -> 59.6 mm
- net +6-8V: track 32.8 -> 23.6 mm
- net /CAN LOW: track 84.0 -> 76.9 mm
- net +12V: track 53.8 -> 57.6 mm
- net Net-(R13-Pad2): track 4.33 -> 6.41 mm
- net GND: track 36.5 -> 38.5 mm
Other:
- board text added: "12V PROT"
- board text added: "3A"
- board text added: "4A"
- board text added: "5V Regulator"
- board text added: "Buck Converter"
- board text added: "CAN Transceiver"
- board text added: "CAN_H"
- board text added: "CAN_L"
- board text added: "Input Protection"
- board text added: "{dblquote}Bahh who needs to breadboard a circuit anyway?{dblquote} Kaboom"
- board text removed: "HIGH"
- board text removed: "LOW"

Commit message: Rev1.1 Started
Rev1.1
Connections:
- U3 pad 3V3R: unconnected-(U3-3V3-Pad3V3R) -> +3.3V
- U4 pad 5: unconnected-(U4-VIO-Pad5) -> +3.3V
Routing:
- net +3.3V: track 0.00 -> 43.4 mm
Changed lines of the file:
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@@
 			(layer "F.SilkS")
 		)
-		(fp_text user "REV 1 - OCT 2026"
+		(fp_text user "REV 1.1 - OCT 26"
 			(at -14.75 6.25 0)
 			(unlocked yes)
@@
 			(layers "F.Cu" "F.Mask" "F.Paste")
 			(roundrect_rratio 0.25)
-			(net "unconnected-(U4-VIO-Pad5)")
+			(net "+3.3V")
 			(pinfunction "VIO_5")
-			(pintype "power_in+no_connect")
+			(pintype "power_in")
 		)
 		(pad "6" smd roundrect
@@
 			(layers "*.Cu" "*.Mask")
 			(remove_unused_layers no)
-			(net "unconnected-(U3-3V3-Pad3V3R)")
+			(net "+3.3V")
 			(pinfunction "3V3_3V3R")
-			(pintype "power_in+no_connect")
+			(pintype "power_in")
 		)
 		(pad "4" thru_hole circle
@@
 	)
 	(segment
-		(start 144.135 63)
-		(end 145.3 63)
+		(start 145.5 63.2)
+		(end 145.905 63.605)
 		(width 0.2)
 		(layer "F.Cu")
@@
 	(segment
 		(start 145.905 63.605)
-		(end 145.3 63)
+		(end 145.905 68.289999)
 		(width 0.2)
 		(layer "F.Cu")
@@
 	)
 	(segment
-		(start 158.0425 80.427499)
-		(end 145.905 68.289999)
+		(start 142.265 64.87)
+		(end 143.935 63.2)
 		(width 0.2)
 		(layer "F.Cu")
@@
 	)
 	(segment
-		(start 145.905 68.289999)
-		(end 145.905 63.605)
+		(start 143.935 63.2)
+		(end 145.5 63.2)
 		(width 0.2)
 		(layer "F.Cu")
@@
 	)
 	(segment
-		(start 142.265 64.87)
-		(end 144.135 63)
+		(start 145.905 68.289999)
+		(end 158.0425 80.427499)
 		(width 0.2)
 		(layer "F.Cu")
@@
 		(net "Net-(D8-K)")
 	)
+	(segment
+		(start 146.30637 62.7)
+		(end 147.345 63.73863)
+		(width 0.2)
+		(layer "F.Cu")
+		(net "+3.3V")
+	)
+	(segment
+		(start 141.7 62.7)
+		(end 146.30637 62.7)
+		(width 0.2)
+		(layer "F.Cu")
+		(net "+3.3V")
+	)
+	(segment
+		(start 162.9925 84.237499)
+		(end 162.3925 84.837499)
+		(width 0.2)
+		(layer "F.Cu")
+		(net "+3.3V")
+	)
+	(segment
+		(start 162.3925 84.837499)
+		(end 155.637499 84.837499)
+		(width 0.2)
+		(layer "F.Cu")
+		(net "+3.3V")
+	)
+	(segment
+		(start 140.825 63.575)
+		(end 141.7 62.7)
+		(width 0.2)
+		(layer "F.Cu")
+		(net "+3.3V")
+	)
+	(segment
+		(start 147.345 63.73863)
+		(end 147.345 64.87)
+		(width 0.2)
+		(layer "F.Cu")
+		(net "+3.3V")
+	)
+	(segment
+		(start 140.825 70.025)
+		(end 140.825 63.575)
+		(width 0.2)
+		(layer "F.Cu")
+		(net "+3.3V")
+	)
+	(segment
+		(start 155.637499 84.837499)
+		(end 140.825 70.025)
+		(width 0.2)
+		(layer "F.Cu")
+		(net "+3.3V")
+	)
 	(zone
